File: eagle-files/Attiny programmer shield.sch (EAGLE design)
At the start: 16 parts, among them IC1 attiny10/11/12/13/15/22/25/45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, IC2 attiny24/44/84, IC3 attiny2313/4313

Commit message: .
Parts:
- removed JP1: PROG-mode, pinhead:PINHD-1X2
- added C2, C4: 100nF, rcl:C-EU050-025X075
- added S2: prog-mode, ccr-lib:SWITCH-SPDT_9.0X4.0MM
- CON1: value AVR-ISP-6 -> ICSP
- R1: value 10kΩ -> 10k
- R2, R3, R4: value 270Ω -> 270; device resistor:R-EU_0207/7 -> resistor:R-EU_0204/5
- U$1: device adafruit:ARDUINO-BPLACE -> ccr-lib:ARDUINO-UNO_R3
- renumbered ICSP1 to CON1, LED1 to D1, LED2 to D2, LED3 to D3
Connections:
- net +UB: now also C2.2, C4.2
- net GND: now also C2.1, C4.1
- net N$1: now also S2.S; no longer JP1.1
- net N$19: now also S2.P, U$1.RESET; no longer JP1.2, U$1./RESET
Other:
- note added: "S2 (prog-mode selector) open : load sketch to Arduino closed : load sketch to an attiny µ-controller"
- note removed: "JP1 (prog-mode selector) open : load sketch to Arduino closed : load sketch to an attiny µ-controller"
- moved on the sheet: C3
